Commit message: feat: robotics structures rework

File: robot/RPR_yyz_renamed.urdf (robot description, URDF)
Before this commit: robot RPR, 5 links, 4 joints
Links:
- removed link Link4
- added link Link1, mass 0; visual box size=0.06 0.06 0.09; visual cylinder length=0.4 radius=0.02
- link Link2: mass 1 -> 0; geometry visual box size=0.03 0.03 0.3; visual cylinder length=0.06 radius=0.03
- link Link3: mass 1 -> 0; geometry visual cylinder length=0.16 radius=0.02
- link base_link: mass 1 -> 0
Joints:
- removed joint ee_link
- added joint JointEE: type fixed, parent Link3, child ee, origin xyz=0.16 0 0 rpy=0 1.57 0
- joint Joint1: child Link2 -> Link1
- joint Joint2: child Link3 -> Link2; parent Link2 -> Link1
- joint Joint3: child Link4 -> Link3; parent Link3 -> Link2
